File: S72forGL516_Template.kicad_pcb (KiCad board)
At the start: 2 copper layers, 314.4 x 98.8 mm, 89 parts, among them J10 Conn_01x01, J11 Conn_01x01, J12 Conn_01x01, J13 Conn_01x01, J14 Conn_01x01, J15 Conn_01x01, J16 Conn_01x01, J17 Conn_01x01, J2 Conn_01x01, J3 Conn_01x01, J4 Conn_01x01, J5 Conn_01x01, J6 Conn_01x01, J7 Conn_01x01, J8 Conn_01x01, J9 Conn_01x01, SW1 SW_PUSH, SW10 SW_PUSH, SW11 SW_PUSH, SW12 SW_PUSH, SW13 SW_PUSH, SW14 SW_PUSH, SW15 SW_PUSH, SW16 SW_PUSH, SW17 SW_PUSH, SW18 SW_PUSH, SW19 SW_PUSH, SW2 KEY_SWITCH, SW20 SW_PUSH, SW21 SW_PUSH, SW22 SW_PUSH, SW23 SW_PUSH, SW24 SW_PUSH, SW25 SW_PUSH, SW26 SW_PUSH, SW27 SW_PUSH, SW28 SW_PUSH, SW29 SW_PUSH, SW3 SW_PUSH, SW30 SW_PUSH, SW31 SW_PUSH, SW32 SW_PUSH, SW33 SW_PUSH, SW34 SW_PUSH, SW35 SW_PUSH, SW36 SW_PUSH, SW37 SW_PUSH, SW38 SW_PUSH, SW39 SW_PUSH, SW4 KEY_SWITCH, SW40 SW_PUSH, SW41 SW_PUSH, SW42 SW_PUSH, SW43 SW_PUSH, SW44 SW_PUSH, SW45 SW_PUSH, SW46 SW_PUSH, SW47 SW_PUSH, SW48 SW_PUSH, SW49 SW_PUSH, SW5 SW_PUSH, SW50 SW_PUSH, SW51 SW_PUSH, SW52 SW_PUSH, SW53 SW_PUSH, SW54 SW_PUSH, SW55 SW_PUSH, SW56 SW_PUSH, SW57 SW_PUSH, SW58 SW_PUSH, SW59 SW_PUSH, SW6 SW_PUSH, SW60 SW_PUSH, SW61 SW_PUSH, SW62 SW_PUSH, SW63 SW_PUSH, SW64 SW_PUSH, SW65 SW_PUSH, SW66 KEY_SWITCH, SW67 SW_PUSH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

Commit message: スイッチプレート作ってみる
Parts:
- removed the SW10 at (52.4, 104.8)
- removed the SW20 at (95.2, 104.8)
- removed the SW25 at (116.7, 104.8)
- removed the SW40 at (178.6, 104.8)
- removed the SW45 at (200.0, 104.8)
- removed the SW50 at (221.5, 104.8)
- removed the SW55 at (245.3, 104.8)
- added SW66: SW_PUSH, kbd_SW_Hole:SW_Hole_1u, F.Cu at (157.2, 104.8)
- added SW67: SW_PUSH, kbd_SW_Hole:SW_Hole_1u, F.Cu at (176.2, 104.8)
- added SW69: KEY_SWITCH, kbd_SW_Hole:SW_Hole_1.25u, F.Cu at (235.7, 104.8)
- added SW70: KEY_SWITCH, kbd_SW_Hole:SW_Hole_1.5u, F.Cu at (261.9, 104.8)
- added SW71: KEY_SWITCH, kbd_SW_Hole:SW_Hole_1.5u, F.Cu at (290.5, 104.8)
- added SW72: SW_PUSH, kbd_SW_Hole:SW_Hole_1u, F.Cu at (314.3, 104.8)
- SW63: footprint kbd_SW_Hole:SW_Hole_1u -> kbd_SW_Hole:SW_Hole_1.25u
- SW68: value SW_PUSH -> KEY_SWITCH; footprint kbd_SW_Hole:SW_Hole_1u -> kbd_SW_Hole:SW_Hole_2u
- moved SW1 285.8 mm to (28.6, 28.6)
- moved SW17 285.8 mm to (28.6, 47.6)
- moved SW32 285.8 mm to (28.6, 66.7)
- moved SW46 285.8 mm to (28.6, 85.7)
- moved SW60 285.8 mm to (28.6, 104.8)
- moved SW63 178.6 mm to (97.6, 104.8)
- moved SW68 90.5 mm to (204.8, 104.8), turned to 180 degrees
- moved SW59 38.1 mm to (307.2, 85.7)
- moved J14 19.1 mm to (253.4, 120.2)
- moved SW10 19.1 mm to (200.0, 28.6)
- moved SW12 19.1 mm to (238.1, 28.6)
- moved SW13 19.1 mm to (257.2, 28.6)
- moved SW14 19.1 mm to (276.2, 28.6)
- moved SW16 19.1 mm to (314.3, 28.6)
- moved SW23 19.1 mm to (152.4, 47.6)
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- renumbered SW69 to SW1, SW41 to SW10, SW46 to SW11, SW51 to SW12, SW56 to SW13, SW59 to SW14, SW64 to SW15, SW65 to SW16, SW70 to SW17, SW2 to SW18, SW7 to SW19, SW1 to SW2, SW12 to SW20, SW17 to SW21, SW27 to SW23, SW32 to SW24, SW37 to SW25, SW42 to SW26, SW47 to SW27, SW52 to SW28, SW57 to SW29, SW6 to SW3, SW60 to SW30, SW66 to SW31, SW71 to SW32, SW3 to SW33, SW8 to SW34, SW13 to SW35, SW18 to SW36, SW23 to SW37, SW28 to SW38, SW33 to SW39, SW11 to SW4, SW38 to SW40, SW43 to SW41, SW48 to SW42, SW53 to SW43, SW58 to SW44, SW61 to SW45, SW72 to SW46, SW4 to SW47, SW9 to SW48, SW14 to SW49, SW16 to SW5, SW19 to SW50, SW24 to SW51, SW29 to SW52, SW34 to SW53, SW39 to SW54, SW44 to SW55, SW49 to SW56, SW54 to SW57, SW67 to SW58, SW62 to SW59, SW21 to SW6, SW73 to SW60, SW5 to SW61, SW15 to SW62, SW30 to SW64, SW35 to SW65, SW26 to SW7, SW31 to SW8, SW36 to SW9
Other:
- net class Default removed

Commit message: フットプリントを配置
Parts:
- removed J10, J11, J12, J13, J14, J15, J16, J17, J8, J9: Conn_01x01, kbd_Hole:m2_Screw_Hole_Fab
- removed J2, J3, J4, J5, J6, J7: Conn_01x01, kbd_Hole:m2_Screw_Hole_EdgeCuts
- added D1: D, kbd_Parts:Diode_TH_SMD, F.Cu at (38.1, 33.3)
- added D10: D, kbd_Parts:Diode_TH_SMD, F.Cu at (207.2, 31.0)
- added D11: D, kbd_Parts:Diode_TH_SMD, F.Cu at (226.2, 31.0)
- added D12: D, kbd_Parts:Diode_TH_SMD, F.Cu at (245.3, 31.0)
- added D13: D, kbd_Parts:Diode_TH_SMD, F.Cu at (264.3, 31.0)
- added D14: D, kbd_Parts:Diode_TH_SMD, F.Cu at (283.4, 31.0)
- added D15: D, kbd_Parts:Diode_TH_SMD, F.Cu at (303.0, 29.7)
- added D16: D, kbd_Parts:Diode_TH_SMD, F.Cu at (322.1, 29.7)
- added D17: D, kbd_Parts:Diode_TH_SMD, F.Cu at (35.7, 50.0)
- added D18: D, kbd_Parts:Diode_TH_SMD, F.Cu at (59.5, 50.0)
- added D19: D, kbd_Parts:Diode_TH_SMD, F.Cu at (83.3, 50.0)
- added D2: D, kbd_Parts:Diode_TH_SMD, F.Cu at (54.8, 31.0)
- added D20: D, kbd_Parts:Diode_TH_SMD, F.Cu at (102.4, 50.0)
- added D21: D, kbd_Parts:Diode_TH_SMD, F.Cu at (121.4, 50.0)
- added D22: D, kbd_Parts:Diode_TH_SMD, F.Cu at (140.5, 50.0)
- added D23: D, kbd_Parts:Diode_TH_SMD, F.Cu at (159.5, 50.0)
- added D24: D, kbd_Parts:Diode_TH_SMD, F.Cu at (178.6, 50.0)
- added D25: D, kbd_Parts:Diode_TH_SMD, F.Cu at (197.6, 50.0)
- added D26: D, kbd_Parts:Diode_TH_SMD, F.Cu at (216.7, 50.0)
- added D27: D, kbd_Parts:Diode_TH_SMD, F.Cu at (235.7, 50.0)
- added D28: D, kbd_Parts:Diode_TH_SMD, F.Cu at (254.8, 50.0)
- added D29: D, kbd_Parts:Diode_TH_SMD, F.Cu at (273.8, 50.0)
- added D3: D, kbd_Parts:Diode_TH_SMD, F.Cu at (73.8, 31.0)
- added D30: D, kbd_Parts:Diode_TH_SMD, F.Cu at (292.9, 50.0)
- added D31: D, kbd_Parts:Diode_TH_SMD, F.Cu at (319.1, 59.5)
- added D32: D, kbd_Parts:Diode_TH_SMD, F.Cu at (35.7, 69.1)
- added D33: D, kbd_Parts:Diode_TH_SMD, F.Cu at (61.9, 69.1)
- added D34: D, kbd_Parts:Diode_TH_SMD, F.Cu at (88.1, 69.1)
- added D35: D, kbd_Parts:Diode_TH_SMD, F.Cu at (107.2, 69.1)
- added D36: D, kbd_Parts:Diode_TH_SMD, F.Cu at (126.2, 69.1)
- added D37: D, kbd_Parts:Diode_TH_SMD, F.Cu at (145.3, 69.1)
- added D38: D, kbd_Parts:Diode_TH_SMD, F.Cu at (164.3, 69.1)
- added D39: D, kbd_Parts:Diode_TH_SMD, F.Cu at (183.4, 69.1)
- added D4: D, kbd_Parts:Diode_TH_SMD, F.Cu at (92.9, 31.0)
- added D40: D, kbd_Parts:Diode_TH_SMD, F.Cu at (202.4, 69.1)
- added D41: D, kbd_Parts:Diode_TH_SMD, F.Cu at (221.5, 69.1)
- added D42: D, kbd_Parts:Diode_TH_SMD, F.Cu at (240.5, 69.1)
- added D43: D, kbd_Parts:Diode_TH_SMD, F.Cu at (259.6, 69.1)
- added D44: D, kbd_Parts:Diode_TH_SMD, F.Cu at (278.6, 69.1)
- added D45: D, kbd_Parts:Diode_TH_SMD, F.Cu at (297.7, 69.1)
- added D46: D, kbd_Parts:Diode_TH_SMD, F.Cu at (35.7, 88.1)
- added D47: D, kbd_Parts:Diode_TH_SMD, F.Cu at (66.7, 88.1)
- added D48: D, kbd_Parts:Diode_TH_SMD, F.Cu at (97.6, 88.1)
- added D49: D, kbd_Parts:Diode_TH_SMD, F.Cu at (116.7, 88.1)
- added D5: D, kbd_Parts:Diode_TH_SMD, F.Cu at (111.9, 31.0)
- added D50: D, kbd_Parts:Diode_TH_SMD, F.Cu at (135.7, 88.1)
- added D51: D, kbd_Parts:Diode_TH_SMD, F.Cu at (154.8, 88.1)
- added D52: D, kbd_Parts:Diode_TH_SMD, F.Cu at (173.8, 88.1)
- added D53: D, kbd_Parts:Diode_TH_SMD, F.Cu at (192.9, 88.1)
- added D54: D, kbd_Parts:Diode_TH_SMD, F.Cu at (211.9, 88.1)
- added D55: D, kbd_Parts:Diode_TH_SMD, F.Cu at (231.0, 88.1)
- added D56: D, kbd_Parts:Diode_TH_SMD, F.Cu at (250.0, 88.1)
- added D57: D, kbd_Parts:Diode_TH_SMD, F.Cu at (269.1, 88.1)
- added D58: D, kbd_Parts:Diode_TH_SMD, F.Cu at (288.1, 88.1)
- added D59: D, kbd_Parts:Diode_TH_SMD, F.Cu at (314.3, 88.1)
- added D6: D, kbd_Parts:Diode_TH_SMD, F.Cu at (131.0, 31.0)
- added D60: D, kbd_Parts:Diode_TH_SMD, F.Cu at (35.7, 107.2)
- added D61: D, kbd_Parts:Diode_TH_SMD, F.Cu at (57.1, 107.2)
- added D62: D, kbd_Parts:Diode_TH_SMD, F.Cu at (81.0, 107.2)
- added D63: D, kbd_Parts:Diode_TH_SMD, F.Cu at (104.8, 107.2)
- added D64: D, kbd_Parts:Diode_TH_SMD, F.Cu at (126.2, 107.2)
- added D65: D, kbd_Parts:Diode_TH_SMD, F.Cu at (145.3, 107.2)
- added D66: D, kbd_Parts:Diode_TH_SMD, F.Cu at (164.3, 107.2)
- added D67: D, kbd_Parts:Diode_TH_SMD, F.Cu at (183.4, 107.2)
- added D68: D, kbd_Parts:Diode_TH_SMD, F.Cu at (211.9, 107.2)
- added D69: D, kbd_Parts:Diode_TH_SMD, F.Cu at (242.9, 107.2)
- added D7: D, kbd_Parts:Diode_TH_SMD, F.Cu at (150.0, 31.0)
- added D70: D, kbd_Parts:Diode_TH_SMD, F.Cu at (269.1, 107.2)
- added D71: D, kbd_Parts:Diode_TH_SMD, F.Cu at (297.7, 107.2)
- added D72: D, kbd_Parts:Diode_TH_SMD, F.Cu at (321.5, 107.2)
- added D8: D, kbd_Parts:Diode_TH_SMD, F.Cu at (169.1, 31.0)
- added D9: D, kbd_Parts:Diode_TH_SMD, F.Cu at (188.1, 31.0)
- added J1: Conn_01x02, kbd_Parts:Battery_XH2.5_GL_PCB, F.Cu at (171.4, 19.1)
- added L1: SK6812MINI, kbd_Parts:LED_SK6812MINI-E_BL, F.Cu at (314.3, 32.5)
- added L10: SK6812MINI, kbd_Parts:LED_SK6812MINI-E_BL, F.Cu at (257.2, 33.3)
- added L11: SK6812MINI, kbd_Parts:LED_SK6812MINI-E_BL, F.Cu at (266.7, 52.4)
- added L12: SK6812MINI, kbd_Parts:LED_SK6812MINI-E_BL, F.Cu at (271.5, 71.4)
- added L13: SK6812MINI, kbd_Parts:LED_SK6812MINI-E_BL, F.Cu at (281.0, 90.5)
- added L14: SK6812MINI, kbd_Parts:LED_SK6812MINI-E_BL, F.Cu at (261.9, 109.5)
- added L15: SK6812MINI, kbd_Parts:LED_SK6812MINI-E_BL, F.Cu at (261.9, 90.5)
- added L16: SK6812MINI, kbd_Parts:LED_SK6812MINI-E_BL, F.Cu at (252.4, 71.4)
- added L17: SK6812MINI, kbd_Parts:LED_SK6812MINI-E_BL, F.Cu at (247.7, 52.4)
- added L18: SK6812MINI, kbd_Parts:LED_SK6812MINI-E_BL, F.Cu at (238.1, 33.3)
- added L19: SK6812MINI, kbd_Parts:LED_SK6812MINI-E_BL, F.Cu at (219.1, 33.3)
- added L2: SK6812MINI, kbd_Parts:LED_SK6812MINI-E_BL, F.Cu at (311.9, 61.9)
- added L20: SK6812MINI, kbd_Parts:LED_SK6812MINI-E_BL, F.Cu at (228.6, 52.4)
- added L21: SK6812MINI, kbd_Parts:LED_SK6812MINI-E_BL, F.Cu at (233.4, 71.4)
- added L22: SK6812MINI, kbd_Parts:LED_SK6812MINI-E_BL, F.Cu at (242.9, 90.5)
- added L23: SK6812MINI, kbd_Parts:LED_SK6812MINI-E_BL, F.Cu at (235.7, 109.5)
- added L24: SK6812MINI, kbd_Parts:LED_SK6812MINI-E_BL, F.Cu at (223.8, 90.5)
- added L25: SK6812MINI, kbd_Parts:LED_SK6812MINI-E_BL, F.Cu at (214.3, 71.4)
- added L26: SK6812MINI, kbd_Parts:LED_SK6812MINI-E_BL, F.Cu at (209.6, 52.4)
- added L27: SK6812MINI, kbd_Parts:LED_SK6812MINI-E_BL, F.Cu at (200.0, 33.3)
- added L28: SK6812MINI, kbd_Parts:LED_SK6812MINI-E_BL, F.Cu at (181.0, 33.3)
- added L29: SK6812MINI, kbd_Parts:LED_SK6812MINI-E_BL, F.Cu at (190.5, 52.4)
- added L3: SK6812MINI, kbd_Parts:LED_SK6812MINI-E_BL, F.Cu at (307.2, 90.5)
- added L30: SK6812MINI, kbd_Parts:LED_SK6812MINI-E_BL, F.Cu at (195.3, 71.4)
- added L31: SK6812MINI, kbd_Parts:LED_SK6812MINI-E_BL, F.Cu at (204.8, 90.5)
- added L32: SK6812MINI, kbd_Parts:LED_SK6812MINI-E_BL, F.Cu at (204.8, 109.5)
- added L33: SK6812MINI, kbd_Parts:LED_SK6812MINI-E_BL, F.Cu at (185.7, 90.5)
- added L34: SK6812MINI, kbd_Parts:LED_SK6812MINI-E_BL, F.Cu at (176.2, 71.4)
- added L35: SK6812MINI, kbd_Parts:LED_SK6812MINI-E_BL, F.Cu at (171.4, 52.4)
- added L36: SK6812MINI, kbd_Parts:LED_SK6812MINI-E_BL, F.Cu at (161.9, 33.3)
- added L37: SK6812MINI, kbd_Parts:LED_SK6812MINI-E_BL, F.Cu at (142.9, 33.3)
- added L38: SK6812MINI, kbd_Parts:LED_SK6812MINI-E_BL, F.Cu at (152.4, 52.4)
- added L39: SK6812MINI, kbd_Parts:LED_SK6812MINI-E_BL, F.Cu at (157.2, 71.4)
- added L4: SK6812MINI, kbd_Parts:LED_SK6812MINI-E_BL, F.Cu at (314.3, 109.5)
- added L40: SK6812MINI, kbd_Parts:LED_SK6812MINI-E_BL, F.Cu at (166.7, 90.5)
- added L41: SK6812MINI, kbd_Parts:LED_SK6812MINI-E_BL, F.Cu at (176.2, 109.5)
- added L42: SK6812MINI, kbd_Parts:LED_SK6812MINI-E_BL, F.Cu at (157.2, 109.5)
- added L43: SK6812MINI, kbd_Parts:LED_SK6812MINI-E_BL, F.Cu at (147.6, 90.5)
- added L44: SK6812MINI, kbd_Parts:LED_SK6812MINI-E_BL, F.Cu at (138.1, 71.4)
- added L45: SK6812MINI, kbd_Parts:LED_SK6812MINI-E_BL, F.Cu at (133.3, 52.4)
- added L46: SK6812MINI, kbd_Parts:LED_SK6812MINI-E_BL, F.Cu at (123.8, 33.3)
- added L47: SK6812MINI, kbd_Parts:LED_SK6812MINI-E_BL, F.Cu at (104.8, 33.3)
- added L48: SK6812MINI, kbd_Parts:LED_SK6812MINI-E_BL, F.Cu at (114.3, 52.4)
- added L49: SK6812MINI, kbd_Parts:LED_SK6812MINI-E_BL, F.Cu at (119.1, 71.4)
- added L5: SK6812MINI, kbd_Parts:LED_SK6812MINI-E_BL, F.Cu at (290.5, 109.5)
- added L50: SK6812MINI, kbd_Parts:LED_SK6812MINI-E_BL, F.Cu at (128.6, 90.5)
- added L51: SK6812MINI, kbd_Parts:LED_SK6812MINI-E_BL, F.Cu at (138.1, 109.5)
- added L52: SK6812MINI, kbd_Parts:LED_SK6812MINI-E_BL, F.Cu at (119.1, 109.5)
- added L53: SK6812MINI, kbd_Parts:LED_SK6812MINI-E_BL, F.Cu at (109.5, 90.5)
- added L54: SK6812MINI, kbd_Parts:LED_SK6812MINI-E_BL, F.Cu at (100.0, 71.4)
- added L55: SK6812MINI, kbd_Parts:LED_SK6812MINI-E_BL, F.Cu at (95.2, 52.4)
- added L56: SK6812MINI, kbd_Parts:LED_SK6812MINI-E_BL, F.Cu at (85.7, 33.3)
- added L57: SK6812MINI, kbd_Parts:LED_SK6812MINI-E_BL, F.Cu at (66.7, 33.3)
- added L58: SK6812MINI, kbd_Parts:LED_SK6812MINI-E_BL, F.Cu at (76.2, 52.4)
- added L59: SK6812MINI, kbd_Parts:LED_SK6812MINI-E_BL, F.Cu at (81.0, 71.4)
- added L6: SK6812MINI, kbd_Parts:LED_SK6812MINI-E_BL, F.Cu at (290.5, 71.4)
- added L60: SK6812MINI, kbd_Parts:LED_SK6812MINI-E_BL, F.Cu at (90.5, 90.5)
- added L61: SK6812MINI, kbd_Parts:LED_SK6812MINI-E_BL, F.Cu at (97.6, 109.5)
- added L62: SK6812MINI, kbd_Parts:LED_SK6812MINI-E_BL, F.Cu at (73.8, 109.5)
- added L63: SK6812MINI, kbd_Parts:LED_SK6812MINI-E_BL, F.Cu at (59.5, 90.5)
- added L64: SK6812MINI, kbd_Parts:LED_SK6812MINI-E_BL, F.Cu at (54.8, 71.4)
- added L65: SK6812MINI, kbd_Parts:LED_SK6812MINI-E_BL, F.Cu at (52.4, 52.4)
- added L66: SK6812MINI, kbd_Parts:LED_SK6812MINI-E_BL, F.Cu at (50.0, 109.5)
- added L67: SK6812MINI, kbd_Parts:LED_SK6812MINI-E_BL, F.Cu at (47.6, 33.3)
- added L68: SK6812MINI, kbd_Parts:LED_SK6812MINI-E_BL, F.Cu at (28.6, 52.4)
- added L69: SK6812MINI, kbd_Parts:LED_SK6812MINI-E_BL, F.Cu at (28.6, 71.4)
- added L7: SK6812MINI, kbd_Parts:LED_SK6812MINI-E_BL, F.Cu at (285.8, 52.4)
- added L70: SK6812MINI, kbd_Parts:LED_SK6812MINI-E_BL, F.Cu at (28.6, 90.5)
- added L71: SK6812MINI, kbd_Parts:LED_SK6812MINI-E_BL, F.Cu at (28.6, 109.5)
- added L8: SK6812MINI, kbd_Parts:LED_SK6812MINI-E_BL, F.Cu at (295.3, 32.5)
- added L9: SK6812MINI, kbd_Parts:LED_SK6812MINI-E_BL, F.Cu at (276.2, 33.3)
- added SW73: SW_PUSH, kbd_Parts:ResetSW, F.Cu at (266.7, 38.1)
- added U1: BLEMicroPro, kbd_Parts:Micon_BMP_GL, F.Cu at (307.2, 27.9)
- SW1: value SW_PUSH -> RotaryEncoder_Switch; footprint kbd_SW_Hole:SW_Hole_1u -> kbd_Parts:RotaryEncoder_EC12E
- SW10, SW11, SW12, SW13, SW14, SW15, SW16, SW17, SW19, SW2, SW20, SW21, SW22, SW23, SW24, SW25, SW26, SW27, SW28, SW29, SW3, SW30, SW32, SW34, SW35, SW36, SW37, SW38, SW39, SW4, SW40, SW41, SW42, SW43, SW44, SW45, SW46, SW48, SW49, SW5, SW50, SW51, SW52, SW53, SW54, SW55, SW56, SW57, SW58, SW6, SW60, SW64, SW65, SW66, SW67, SW7, SW72, SW8, SW9: footprint kbd_SW_Hole:SW_Hole_1u -> kbd_SW:CherryMX_Hotswap_1u
- SW18, SW70, SW71: value KEY_SWITCH -> SW_PUSH; footprint kbd_SW_Hole:SW_Hole_1.5u -> kbd_SW:CherryMX_Hotswap_1.5u
- SW31: value KEY_SWITCH -> SW_PUSH; footprint kbd_SW_Hole:SW_Hole_2u -> kbd_SW:CherryMX_Hotswap_ISO_Rev
- SW33, SW59: footprint kbd_SW_Hole:SW_Hole_1.75u -> kbd_SW:CherryMX_Hotswap_1.75u
- SW47: value KEY_SWITCH -> SW_PUSH; footprint kbd_SW_Hole:SW_Hole_2.25u -> kbd_SW:CherryMX_Hotswap_2.25u_Rev
- SW61, SW62, SW63: footprint kbd_SW_Hole:SW_Hole_1.25u -> kbd_SW:CherryMX_Hotswap_1.25u
- SW68: value KEY_SWITCH -> SW_PUSH; footprint kbd_SW_Hole:SW_Hole_2u -> kbd_SW:CherryMX_Hotswap_2u_Rev
- SW69: value KEY_SWITCH -> SW_PUSH; footprint kbd_SW_Hole:SW_Hole_1.25u -> kbd_SW:CherryMX_Hotswap_1.25u
- turned SW1 to -90 degrees
- turned SW31 to 90 degrees
Other:
- board size 314.4 x 98.8 mm -> 304.4 x 98.8 mm
- board text removed: "Do not place switches to the Right of this line."
- board text removed: "Do not place switches to the left of this line."
- board text removed: "Put the ProMicro between here and there."
- board text removed: "USB connector to the right.▶"
- board text removed: "▲"
- board text removed: "◀USB connector to the left."
